File: ESP8266getway/untitled.brd (EAGLE design)
At the start: 100 x 80 mm, 18 parts, among them IC1 LM1117MP-3.3

Commit message: 2092017
Parts:
- moved R4 6.75 mm to (36.8, 48.3)
- moved LED3 5.08 mm to (26.0, 55.9)
- moved JP7 3.18 mm to (26.0, 60.3)
- moved R1 2.62 mm to (32.4, 62.2)
- moved R5 2.62 mm to (32.4, 54.0)
Connections:
- removed net N$14: R1.1, U$1.GPIO5
- new net N$25: R1.1, U$1.GPIO4
- net +3V3: no longer R4.1
- net GND: now also R4.2
- net N$1: now also U$1.GPIO5; no longer U$1.GPIO4
- net N$11: now also R5.1; no longer JP7.1, R4.2
- net N$2: now also R4.1
- net N$3: now also JP7.1; no longer R5.1
Routing:
- net N$3: track 5.25 -> 13.9 mm
- net N$11: track 14.0 -> 6.11 mm
- net N$25: track 0.00 -> 5.79 mm
- net N$14: track 4.93 -> 0.00 mm
- net N$1: track 70.6 -> 66.4 mm
- net +3V3: track 52.4 -> 48.9 mm
- net N$12: track 7.35 -> 4.92 mm
- net N$13: track 7.43 -> 5.18 mm
- net GND: track 125.2 -> 126.1 mm

Commit message: 07092017
Parts:
- C1, C2: value (none) -> 47uf
- R1, R3, R5: value (none) -> 1k
- R2, R4: value (none) -> 10k
- moved C1 5.08 mm to (47.6, 42.5)
- moved C3 5.08 mm to (52.7, 43.2)
- moved JP2 1.80 mm to (27.3, 50.8)
- moved LED2 1.80 mm to (27.3, 63.5), turned to 0 degrees
- moved JP4 1.42 mm to (31.8, 69.2)
- moved JP7 1.42 mm to (27.3, 59.7)
- moved R5 1.27 mm to (33.7, 54.0)
- moved LED3 1.27 mm to (27.3, 55.9), turned to 0 degrees
- moved LED1 0.90 mm to (62.2, 62.2), turned to 270 degrees
- moved R1 0.64 mm to (33.0, 62.2)
Connections:
- net +3V3: now also LED1.A, LED2.A, LED3.A
- net GND: no longer LED1.K, LED2.K, LED3.K
- net N$12: now also LED3.K; no longer LED3.A
- net N$13: now also LED2.K; no longer LED2.A
- net N$8: now also LED1.K; no longer LED1.A
Routing:
- net +3V3: track 48.9 -> 116.7 mm, vias 2 -> 4
- net GND: track 126.1 -> 141.8 mm, vias 4 -> 7
- net +5V: track 5.78 -> 3.98 mm
- net N$11: track 6.11 -> 4.84 mm
- net N$3: track 13.9 -> 12.7 mm
- net N$13: track 5.18 -> 4.02 mm
- net N$25: track 5.79 -> 5.16 mm
- net N$8: track 3.89 -> 3.39 mm
